Commit message: add husky 2020.01.29

File: DynamicMotionPlanning/husky/husky_description/urdf/husky.urdf.xacro (robot description, xacro)
@@ -1,3 +1,7 @@
-<?xml version="1.0"?>
+<?xml version="1.0" ?>
+<!-- =================================================================================== -->
+<!-- |    This document was autogenerated by xacro from /home/mrjohd/MotionPlanning_ws/src/DynamicMotionPlanning/husky/husky_description/urdf/husky.urdf.xacro | -->
+<!-- |    EDITING THIS FILE BY HAND IS NOT RECOMMENDED                                 | -->
+<!-- =================================================================================== -->
 <!--
 Software License Agreement (BSD)
@@ -22,34 +26,6 @@
 -->
 <robot name="husky" xmlns:xacro="http://ros.org/wiki/xacro">
-  <xacro:arg name="laser_enabled" default="false" />
-  <xacro:arg name="laser_xyz" default="$(optenv HUSKY_LMS1XX_XYZ 0.2206 0.0 0.00635)" />
-  <xacro:arg name="laser_rpy" default="$(optenv HUSKY_LMS1XX_RPY 0.0 0.0 0.0)" />
-  <xacro:arg name="kinect_enabled" default="false" />
-  <xacro:arg name="kinect_xyz" default="$(optenv HUSKY_KINECT_XYZ 0 0 0)" />
-  <xacro:arg name="kinect_rpy" default="$(optenv HUSKY_KINECT_RPY 0 0.18 3.14)" />
-  <xacro:property name="husky_front_bumper_extend" value="$(optenv HUSKY_FRONT_BUMPER_EXTEND 0)" />
-  <xacro:property name="husky_rear_bumper_extend" value="$(optenv HUSKY_REAR_BUMPER_EXTEND 0)" />
-  <xacro:arg name="robot_namespace" default="/" />
-  <xacro:arg name="urdf_extras" default="empty.urdf" />
-  <!-- Included URDF/XACRO Files -->
-  <xacro:include filename="$(find husky_description)/urdf/decorations.urdf.xacro" />
-  <xacro:include filename="$(find husky_description)/urdf/wheel.urdf.xacro" />
-  <xacro:include filename="$(find husky_description)/urdf/accessories/kinect_camera.urdf.xacro"/>
-  <xacro:include filename="$(find husky_description)/urdf/accessories/sick_lms1xx_mount.urdf.xacro"/>
-  <xacro:include filename="$(find husky_description)/urdf/accessories/sensor_arch.urdf.xacro"/>
-  <xacro:property name="M_PI" value="3.14159"/>
-  <!-- Base Size -->
-  <xacro:property name="base_x_size" value="0.98740000" />
-  <xacro:property name="base_y_size" value="0.57090000" />
-  <xacro:property name="base_z_size" value="0.24750000" />
-  <!-- Wheel Mounting Positions -->
-  <xacro:property name="wheelbase" value="0.5120" />
-  <xacro:property name="track" value="0.5708" />
-  <xacro:property name="wheel_vertical_offset" value="0.03282" />
-  <!-- Wheel Properties -->
-  <xacro:property name="wheel_length" value="0.1143" />
-  <xacro:property name="wheel_radius" value="0.1651" />
-  <!-- Base link is the center of the robot's bottom plate -->
-  <link name="world" />
+    <!-- Base link is the center of the robot's bottom plate -->
+    <!-- <link name="world" />
   <joint name="odom_joint" type="fixed">
           <parent link="world"/>
@@ -57,5 +33,5 @@
   </joint>
   <link name="odom">
-      <inertial>
+<inertial>
               <mass value="1" />
               <origin xyz="0.0 0.0 0.0" rpy="0 0 0" />
@@ -73,5 +49,5 @@
   </joint>
   <link name="base_x_link">
-        <inertial>
+<inertial>
                 <mass value="1" />
                 <origin xyz="0 0 0.0" />
@@ -89,5 +65,5 @@
   </joint>
   <link name="base_y_link">
-        <inertial>
+<inertial>
                 <mass value="1" />
                 <origin xyz="0.0 0.0 0.0" rpy="0 0 0" />
@@ -103,130 +79,409 @@
             <parent link="base_y_link"/>
             <child link="base_link" />
-  </joint>
-  <link name="base_link">
-    <visual>
-      <origin xyz="0 0 0" rpy="0 0 0" />
-      <geometry>
-        <mesh filename="package://husky_description/meshes/base_link.dae" />
-      </geometry>
-    </visual>
-    <collision>
-      <origin xyz="${( husky_front_bumper_extend - husky_rear_bumper_extend ) / 2.0} 0 ${base_z_size/4}" rpy="0 0 0" />
-      <geometry>
-        <box size="${ base_x_size + husky_front_bumper_extend + husky_rear_bumper_extend } ${base_y_size} ${base_z_size/2}"/>
-      </geometry>
-    </collision>
-    <collision>
-      <origin xyz="0 0 ${base_z_size*3/4-0.01}" rpy="0 0 0" />
-      <geometry>
-        <box size="${base_x_size*4/5} ${base_y_size} ${base_z_size/2-0.02}"/>
-      </geometry>
-    </collision>
-  </link>
-  <!-- Base footprint is on the ground under the robot -->
-  <link name="base_footprint"/>
-  <joint name="base_footprint_joint" type="fixed">
-    <origin xyz="0 0 ${wheel_vertical_offset - wheel_radius}" rpy="0 0 0" />
-    <parent link="base_link" />
-    <child link="base_footprint" />
-  </joint>
-  <!-- Interial link stores the robot's inertial information -->
-  <link name="inertial_link">
-    <inertial>
-      <mass value="46.034" />
-      <origin xyz="-0.00065 -0.085 0.062" />
-      <inertia ixx="0.6022" ixy="-0.02364" ixz="-0.1197" iyy="1.7386" iyz="-0.001544" izz="2.0296" />
-    </inertial>
-  </link>
-  <joint name="inertial_joint" type="fixed">
-    <origin xyz="0 0 0" rpy="0 0 0" />
-    <parent link="base_link" />
-    <child link="inertial_link" />
-  </joint>
-  <!-- IMU Link is the standard mounting position for the UM6 IMU.-->
-  <!-- Can be modified with environment variables in /etc/ros/setup.bash -->
-  <link name="imu_link"/>
-  <joint name="imu_joint" type="fixed">
-    <origin xyz="$(optenv HUSKY_IMU_XYZ 0.19 0 0.149)" rpy="$(optenv HUSKY_IMU_RPY 0 -1.5708 3.1416)" />
-    <parent link="base_link" />
-    <child link="imu_link" />
-  </joint>
-  <gazebo reference="imu_link">
-  </gazebo>
-  <!-- Husky wheel macros -->
-  <xacro:husky_wheel wheel_prefix="front_left">
-    <origin xyz="${wheelbase/2} ${track/2} ${wheel_vertical_offset}" rpy="0 0 0" />
-  </xacro:husky_wheel>
-  <xacro:husky_wheel wheel_prefix="front_right">
-    <origin xyz="${wheelbase/2} ${-track/2} ${wheel_vertical_offset}" rpy="0 0 0" />
-  </xacro:husky_wheel>
-  <xacro:husky_wheel wheel_prefix="rear_left">
-    <origin xyz="${-wheelbase/2} ${track/2} ${wheel_vertical_offset}" rpy="0 0 0" />
-  </xacro:husky_wheel>
-  <xacro:husky_wheel wheel_prefix="rear_right">
-    <origin xyz="${-wheelbase/2} ${-track/2} ${wheel_vertical_offset}" rpy="0 0 0" />
-  </xacro:husky_wheel>
-  <xacro:husky_decorate />
-  <xacro:if value="$(arg laser_enabled)">
-    <sick_lms1xx_mount prefix="base"/>
-    <sick_lms1xx frame="base_laser" topic="scan" robot_namespace="$(arg robot_namespace)"/>
-    <joint name="laser_mount_joint" type="fixed">
-      <origin xyz="$(arg laser_xyz)" rpy="$(arg laser_rpy)" />
-      <parent link="top_plate_link" />
-      <child link="base_laser_mount" />
-    </joint>
-  </xacro:if>
-  <xacro:if value="$(arg kinect_enabled)">
-    <xacro:sensor_arch prefix="" parent="top_plate_link">
-      <origin xyz="-0.35 0 0.51" rpy="0 0 -3.14"/>
-    </xacro:sensor_arch>
-    <joint name="kinect_frame_joint" type="fixed">
-      <origin xyz="$(arg kinect_xyz)" rpy="$(arg kinect_rpy)" />
-      <parent link="sensor_arch_mount_link"/>
-      <child link="camera_link"/>
-    </joint>
-    <xacro:kinect_camera prefix="camera" robot_namespace="$(arg robot_namespace)"/>
-  </xacro:if>
-  <gazebo>
-    <plugin name="gazebo_ros_control" filename="libgazebo_ros_control.so">
-      <robotNamespace>$(arg robot_namespace)</robotNamespace>
-    </plugin>
-  </gazebo>
-  <gazebo>
-    <plugin name="imu_controller" filename="libhector_gazebo_ros_imu.so">
-      <robotNamespace>$(arg robot_namespace)</robotNamespace>
-      <updateRate>50.0</updateRate>
-      <bodyName>base_link</bodyName>
-      <topicName>imu/data</topicName>
-      <accelDrift>0.005 0.005 0.005</accelDrift>
-      <accelGaussianNoise>0.005 0.005 0.005</accelGaussianNoise>
-      <rateDrift>0.005 0.005 0.005 </rateDrift>
-      <rateGaussianNoise>0.005 0.005 0.005 </rateGaussianNoise>
-      <headingDrift>0.005</headingDrift>
-      <headingGaussianNoise>0.005</headingGaussianNoise>
-    </plugin>
-  </gazebo>
-  <gazebo>
-    <plugin name="gps_controller" filename="libhector_gazebo_ros_gps.so">
-      <robotNamespace>$(arg robot_namespace)</robotNamespace>
-      <updateRate>40</updateRate>
-      <bodyName>base_link</bodyName>
-      <frameId>base_link</frameId>
-      <topicName>navsat/fix</topicName>
-      <velocityTopicName>navsat/vel</velocityTopicName>
-      <referenceLatitude>49.9</referenceLatitude>
-      <referenceLongitude>8.9</referenceLongitude>
-      <referenceHeading>0</referenceHeading>
-      <referenceAltitude>0</referenceAltitude>
-      <drift>0.0001 0.0001 0.0001</drift>
-    </plugin>
-  </gazebo>
-  <gazebo>
-    <plugin name="husky" filename="libhusky.so"/>
-  </gazebo>
-  <gazebo>
-    <plugin name="planning_scene" filename="libplanning_scene.so"/>
-  </gazebo>
-  <!-- Optional custom includes. -->
-  <xacro:include filename="$(arg urdf_extras)" />
+  </joint> -->
+    <link name="base_link">
+        <visual>
+            <origin rpy="0 0 0" xyz="0 0 0" />
+            <geometry>
+                <mesh filename="package://husky_description/meshes/base_link.dae" />
+            </geometry>
+        </visual>
+        <collision>
+            <origin rpy="0 0 0" xyz="0.0 0 0.061875" />
+            <geometry>
+                <box size="0.9874 0.5709 0.12375" />
+            </geometry>
+        </collision>
+        <collision>
+            <origin rpy="0 0 0" xyz="0 0 0.175625" />
+            <geometry>
+                <box size="0.78992 0.5709 0.10375" />
+            </geometry>
+        </collision>
+        <inertial>
+            <mass value="0.1" />
+            <inertia ixx="0.03" iyy="0.03" izz="0.03" ixy="0.0" ixz="0.0" iyz="0.0" />
+        </inertial>
+    </link>
+    <!-- Base footprint is on the ground under the robot -->
+    <link name="base_footprint" />
+    <joint name="base_footprint_joint" type="fixed">
+        <origin rpy="0 0 0" xyz="0 0 -0.13228" />
+        <parent link="base_link" />
+        <child link="base_footprint" />
+    </joint>
+    <!-- Interial link stores the robot's inertial information -->
+    <link name="inertial_link">
+        <inertial>
+            <mass value="46.034" />
+            <origin xyz="-0.00065 -0.085 0.062" />
+            <inertia ixx="0.6022" ixy="-0.02364" ixz="-0.1197" iyy="1.7386" iyz="-0.001544" izz="2.0296" />
+        </inertial>
+    </link>
+    <joint name="inertial_joint" type="fixed">
+        <origin rpy="0 0 0" xyz="0 0 0" />
+        <parent link="base_link" />
+        <child link="inertial_link" />
+    </joint>
+    <!-- IMU Link is the standard mounting position for the UM6 IMU.-->
+    <!-- Can be modified with environment variables in /etc/ros/setup.bash -->
+    <link name="imu_link" />
+    <joint name="imu_joint" type="fixed">
+        <origin rpy="0 -1.5708 3.1416" xyz="0.19 0 0.149" />
+        <parent link="base_link" />
+        <child link="imu_link" />
+    </joint>
+    <gazebo reference="imu_link" />
+    <link name="front_left_wheel_link">
+        <inertial>
+            <mass value="2.637" />
+            <origin xyz="0 0 0" />
+            <inertia ixx="0.02467" ixy="0" ixz="0" iyy="0.04411" iyz="0" izz="0.02467" />
+        </inertial>
+        <visual>
+            <origin rpy="0 0 0" xyz="0 0 0" />
+            <geometry>
+                <mesh filename="package://husky_description/meshes/wheel.dae" />
+            </geometry>
+        </visual>
+        <collision>
+            <origin rpy="1.570795 0 0" xyz="0 0 0" />
+            <geometry>
+                <cylinder length="0.1143" radius="0.1651" />
+            </geometry>
+        </collision>
+    </link>
+    <gazebo reference="front_left_wheel_link">
+        <mu1 value="1.0" />
+        <mu2 value="1.0" />
+        <kp value="10000000.0" />
+        <kd value="1.0" />
+        <fdir1 value="1 0 0" />
+    </gazebo>
+    <joint name="front_left_wheel" type="continuous">
+        <parent link="base_link" />
+        <child link="front_left_wheel_link" />
+        <origin rpy="0 0 0" xyz="0.256 0.2854 0.03282" />
+        <axis rpy="0 0 0" xyz="0 1 0" />
+    </joint>
+    <transmission name="front_left_wheel_trans" type="SimpleTransmission">
+        <type>transmission_interface/SimpleTransmission</type>
+        <actuator name="front_left_wheel_motor">
+            <mechanicalReduction>1</mechanicalReduction>
+        </actuator>
+        <joint name="front_left_wheel">
+            <hardwareInterface>hardware_interface/VelocityJointInterface</hardwareInterface>
+        </joint>
+    </transmission>
+    <link name="front_right_wheel_link">
+        <inertial>
+            <mass value="2.637" />
+            <origin xyz="0 0 0" />
+            <inertia ixx="0.02467" ixy="0" ixz="0" iyy="0.04411" iyz="0" izz="0.02467" />
+        </inertial>
+        <visual>
+            <origin rpy="0 0 0" xyz="0 0 0" />
+            <geometry>
+                <mesh filename="package://husky_description/meshes/wheel.dae" />
+            </geometry>
+        </visual>
+        <collision>
+            <origin rpy="1.570795 0 0" xyz="0 0 0" />
+            <geometry>
+                <cylinder length="0.1143" radius="0.1651" />
+            </geometry>
+        </collision>
+    </link>
+    <gazebo reference="front_right_wheel_link">
+        <mu1 value="1.0" />
+        <mu2 value="1.0" />
+        <kp value="10000000.0" />
+        <kd value="1.0" />
+        <fdir1 value="1 0 0" />
+    </gazebo>
+    <joint name="front_right_wheel" type="continuous">
+        <parent link="base_link" />
+        <child link="front_right_wheel_link" />
+        <origin rpy="0 0 0" xyz="0.256 -0.2854 0.03282" />
+        <axis rpy="0 0 0" xyz="0 1 0" />
+    </joint>
+    <transmission name="front_right_wheel_trans" type="SimpleTransmission">
+        <type>transmission_interface/SimpleTransmission</type>
+        <actuator name="front_right_wheel_motor">
+            <mechanicalReduction>1</mechanicalReduction>
+        </actuator>
+        <joint name="front_right_wheel">
+            <hardwareInterface>hardware_interface/VelocityJointInterface</hardwareInterface>
+        </joint>
+    </transmission>
+    <link name="rear_left_wheel_link">
+        <inertial>
+            <mass value="2.637" />
+            <origin xyz="0 0 0" />
+            <inertia ixx="0.02467" ixy="0" ixz="0" iyy="0.04411" iyz="0" izz="0.02467" />
+        </inertial>
+        <visual>
+            <origin rpy="0 0 0" xyz="0 0 0" />
+            <geometry>
+                <mesh filename="package://husky_description/meshes/wheel.dae" />
+            </geometry>
+        </visual>
+        <collision>
+            <origin rpy="1.570795 0 0" xyz="0 0 0" />
+            <geometry>
+                <cylinder length="0.1143" radius="0.1651" />
+            </geometry>
+        </collision>
+    </link>
+    <gazebo reference="rear_left_wheel_link">
+        <mu1 value="1.0" />
+        <mu2 value="1.0" />
+        <kp value="10000000.0" />
+        <kd value="1.0" />
+        <fdir1 value="1 0 0" />
+    </gazebo>
+    <joint name="rear_left_wheel" type="continuous">
+        <parent link="base_link" />
+        <child link="rear_left_wheel_link" />
+        <origin rpy="0 0 0" xyz="-0.256 0.2854 0.03282" />
+        <axis rpy="0 0 0" xyz="0 1 0" />
+    </joint>
+    <transmission name="rear_left_wheel_trans" type="SimpleTransmission">
+        <type>transmission_interface/SimpleTransmission</type>
+        <actuator name="rear_left_wheel_motor">
+            <mechanicalReduction>1</mechanicalReduction>
+        </actuator>
+        <joint name="rear_left_wheel">
+            <hardwareInterface>hardware_interface/VelocityJointInterface</hardwareInterface>
+        </joint>
+    </transmission>
+    <link name="rear_right_wheel_link">
+        <inertial>
+            <mass value="2.637" />
+            <origin xyz="0 0 0" />
+            <inertia ixx="0.02467" ixy="0" ixz="0" iyy="0.04411" iyz="0" izz="0.02467" />
+        </inertial>
+        <visual>
+            <origin rpy="0 0 0" xyz="0 0 0" />
+            <geometry>
+                <mesh filename="package://husky_description/meshes/wheel.dae" />
+            </geometry>
+        </visual>
+        <collision>
+            <origin rpy="1.570795 0 0" xyz="0 0 0" />
+            <geometry>
+                <cylinder length="0.1143" radius="0.1651" />
+            </geometry>
+        </collision>
+    </link>
+    <gazebo reference="rear_right_wheel_link">
+        <mu1 value="1.0" />
+        <mu2 value="1.0" />
+        <kp value="10000000.0" />
+        <kd value="1.0" />
+        <fdir1 value="1 0 0" />
+    </gazebo>
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