Commit message: add husky 2020.02.04

File: DynamicMotionPlanning/husky/husky_description/urdf/husky.urdf.xacro (robot description, xacro)
@@ -1,7 +1,3 @@
-<?xml version="1.0" ?>
-<!-- =================================================================================== -->
-<!-- |    This document was autogenerated by xacro from /home/mrjohd/MotionPlanning_ws/src/DynamicMotionPlanning/husky/husky_description/urdf/husky.urdf.xacro | -->
-<!-- |    EDITING THIS FILE BY HAND IS NOT RECOMMENDED                                 | -->
-<!-- =================================================================================== -->
+<?xml version="1.0"?>
 <!--
 Software License Agreement (BSD)
@@ -26,12 +22,51 @@
 -->
 <robot name="husky" xmlns:xacro="http://ros.org/wiki/xacro">
-    <!-- Base link is the center of the robot's bottom plate -->
-    <!-- <link name="world" />
+  <xacro:arg name="laser_enabled" default="true" />
+  <xacro:arg name="laser_xyz" default="$(optenv HUSKY_LMS1XX_XYZ 0.2206 0.0 0.00635)" />
+  <xacro:arg name="laser_rpy" default="$(optenv HUSKY_LMS1XX_RPY 0.0 0.0 0.0)" />
+  <xacro:arg name="kinect_enabled" default="true" />
+  <xacro:arg name="kinect_xyz" default="$(optenv HUSKY_KINECT_XYZ 0 0 0)" />
+  <xacro:arg name="kinect_rpy" default="$(optenv HUSKY_KINECT_RPY 0 0.18 3.14)" />
+  <xacro:property name="husky_front_bumper_extend" value="$(optenv HUSKY_FRONT_BUMPER_EXTEND 0)" />
+  <xacro:property name="husky_rear_bumper_extend" value="$(optenv HUSKY_REAR_BUMPER_EXTEND 0)" />
+  <xacro:arg name="robot_namespace" default="husky" />
+  <xacro:arg name="urdf_extras" default="empty.urdf" />
+  <!-- Included URDF/XACRO Files -->
+  <xacro:include filename="$(find husky_description)/urdf/decorations.urdf.xacro" />
+  <xacro:include filename="$(find husky_description)/urdf/wheel.urdf.xacro" />
+  <xacro:include filename="$(find husky_description)/urdf/accessories/kinect_camera.urdf.xacro"/>
+  <xacro:include filename="$(find husky_description)/urdf/accessories/sick_lms1xx_mount.urdf.xacro"/>
+  <xacro:include filename="$(find husky_description)/urdf/accessories/sensor_arch.urdf.xacro"/>
+  <xacro:property name="M_PI" value="3.14159"/>
+  <!-- Base Size -->
+  <xacro:property name="base_x_size" value="0.98740000" />
+  <xacro:property name="base_y_size" value="0.57090000" />
+  <xacro:property name="base_z_size" value="0.24750000" />
+  <!-- Wheel Mounting Positions -->
+  <xacro:property name="wheelbase" value="0.5120" />
+  <xacro:property name="track" value="0.5708" />
+  <xacro:property name="wheel_vertical_offset" value="0.03282" />
+  <!-- Wheel Properties -->
+  <xacro:property name="wheel_length" value="0.1143" />
+  <xacro:property name="wheel_radius" value="0.1651" />
+  <!-- Base link is the center of the robot's bottom plate -->
+  <link name="world" />
+  <joint name="map_joint" type="fixed">
+          <parent link="world"/>
+          <child link="map" />
+  </joint>
+  <link name="map">
+      <inertial>
+              <mass value="1" />
+              <origin xyz="0.0 0.0 0.0" rpy="0 0 0" />
+              <inertia ixx="0.1" ixy="0.0" ixz="0.0"	iyy="0.1" iyz="0.0" izz="0.1" />
+      </inertial>
+  </link>
   <joint name="odom_joint" type="fixed">
-          <parent link="world"/>
+          <parent link="map"/>
           <child link="odom" />
   </joint>
   <link name="odom">
-<inertial>
+      <inertial>
               <mass value="1" />
               <origin xyz="0.0 0.0 0.0" rpy="0 0 0" />
@@ -49,5 +84,5 @@
   </joint>
   <link name="base_x_link">
-<inertial>
+        <inertial>
                 <mass value="1" />
                 <origin xyz="0 0 0.0" />
@@ -65,5 +100,5 @@
   </joint>
   <link name="base_y_link">
-<inertial>
+        <inertial>
                 <mass value="1" />
                 <origin xyz="0.0 0.0 0.0" rpy="0 0 0" />
@@ -79,409 +114,147 @@
             <parent link="base_y_link"/>
             <child link="base_link" />
+  </joint>
+  <!-- <joint name="odom2base_joint" type="fixed">
+          <parent link="odom"/>
+          <child link="base_link" />
   </joint> -->
-    <link name="base_link">
-        <visual>
-            <origin rpy="0 0 0" xyz="0 0 0" />
-            <geometry>
-                <mesh filename="package://husky_description/meshes/base_link.dae" />
-            </geometry>
-        </visual>
-        <collision>
-            <origin rpy="0 0 0" xyz="0.0 0 0.061875" />
-            <geometry>
-                <box size="0.9874 0.5709 0.12375" />
-            </geometry>
-        </collision>
-        <collision>
-            <origin rpy="0 0 0" xyz="0 0 0.175625" />
-            <geometry>
-                <box size="0.78992 0.5709 0.10375" />
-            </geometry>
-        </collision>
-        <inertial>
-            <mass value="0.1" />
-            <inertia ixx="0.03" iyy="0.03" izz="0.03" ixy="0.0" ixz="0.0" iyz="0.0" />
-        </inertial>
-    </link>
-    <!-- Base footprint is on the ground under the robot -->
-    <link name="base_footprint" />
-    <joint name="base_footprint_joint" type="fixed">
-        <origin rpy="0 0 0" xyz="0 0 -0.13228" />
-        <parent link="base_link" />
-        <child link="base_footprint" />
+  <link name="base_link">
+    <visual>
+      <origin xyz="0 0 0" rpy="0 0 0" />
+      <geometry>
+        <mesh filename="package://husky_description/meshes/base_link.dae" />
+      </geometry>
+    </visual>
+    <collision>
+      <origin xyz="${( husky_front_bumper_extend - husky_rear_bumper_extend ) / 2.0} 0 ${base_z_size/4}" rpy="0 0 0" />
+      <geometry>
+        <box size="${ base_x_size + husky_front_bumper_extend + husky_rear_bumper_extend } ${base_y_size} ${base_z_size/2}"/>
+      </geometry>
+    </collision>
+    <collision>
+      <origin xyz="0 0 ${base_z_size*3/4-0.01}" rpy="0 0 0" />
+      <geometry>
+        <box size="${base_x_size*4/5} ${base_y_size} ${base_z_size/2-0.02}"/>
+      </geometry>
+    </collision>
+  </link>
+  <!-- Base footprint is on the ground under the robot -->
+  <joint name="base_footprint_joint" type="fixed">
+    <origin xyz="0 0 ${wheel_vertical_offset - wheel_radius}" rpy="0 0 0" />
+    <parent link="base_link" />
+    <child link="base_footprint" />
+  </joint>
+  <link name="base_footprint"/>
+  <!-- Interial link stores the robot's inertial information -->
+  <link name="inertial_link">
+    <inertial>
+      <mass value="46.034" />
+      <origin xyz="-0.00065 -0.085 0.062" />
+      <inertia ixx="0.6022" ixy="-0.02364" ixz="-0.1197" iyy="1.7386" iyz="-0.001544" izz="2.0296" />
+    </inertial>
+  </link>
+  <joint name="inertial_joint" type="fixed">
+    <origin xyz="0 0 0" rpy="0 0 0" />
+    <parent link="base_link" />
+    <child link="inertial_link" />
+  </joint>
+  <!-- IMU Link is the standard mounting position for the UM6 IMU.-->
+  <!-- Can be modified with environment variables in /etc/ros/setup.bash -->
+  <link name="imu_link"/>
+  <joint name="imu_joint" type="fixed">
+    <origin xyz="$(optenv HUSKY_IMU_XYZ 0.19 0 0.149)" rpy="$(optenv HUSKY_IMU_RPY 0 -1.5708 3.1416)" />
+    <parent link="base_link" />
+    <child link="imu_link" />
+  </joint>
+  <gazebo reference="imu_link">
+  </gazebo>
+  <!-- Husky wheel macros -->
+  <xacro:husky_wheel wheel_prefix="front_left">
+    <origin xyz="${wheelbase/2} ${track/2} ${wheel_vertical_offset}" rpy="0 0 0" />
+  </xacro:husky_wheel>
+  <xacro:husky_wheel wheel_prefix="front_right">
+    <origin xyz="${wheelbase/2} ${-track/2} ${wheel_vertical_offset}" rpy="0 0 0" />
+  </xacro:husky_wheel>
+  <xacro:husky_wheel wheel_prefix="rear_left">
+    <origin xyz="${-wheelbase/2} ${track/2} ${wheel_vertical_offset}" rpy="0 0 0" />
+  </xacro:husky_wheel>
+  <xacro:husky_wheel wheel_prefix="rear_right">
+    <origin xyz="${-wheelbase/2} ${-track/2} ${wheel_vertical_offset}" rpy="0 0 0" />
+  </xacro:husky_wheel>
+  <xacro:husky_decorate />
+  <xacro:if value="$(arg laser_enabled)">
+    <sick_lms1xx_mount prefix="base"/>
+    <sick_lms1xx frame="base_laser" topic="scan" robot_namespace="$(arg robot_namespace)"/>
+    <joint name="laser_mount_joint" type="fixed">
+      <origin xyz="$(arg laser_xyz)" rpy="$(arg laser_rpy)" />
+      <parent link="top_plate_link" />
+      <child link="base_laser_mount" />
     </joint>
-    <!-- Interial link stores the robot's inertial information -->
-    <link name="inertial_link">
-        <inertial>
-            <mass value="46.034" />
-            <origin xyz="-0.00065 -0.085 0.062" />
-            <inertia ixx="0.6022" ixy="-0.02364" ixz="-0.1197" iyy="1.7386" iyz="-0.001544" izz="2.0296" />
-        </inertial>
-    </link>
-    <joint name="inertial_joint" type="fixed">
-        <origin rpy="0 0 0" xyz="0 0 0" />
-        <parent link="base_link" />
-        <child link="inertial_link" />
+  </xacro:if>
+  <xacro:if value="$(arg kinect_enabled)">
+    <xacro:sensor_arch prefix="" parent="top_plate_link">
+      <origin xyz="-0.35 0 0.51" rpy="0 0 -3.14"/>
+    </xacro:sensor_arch>
+    <joint name="kinect_frame_joint" type="fixed">
+      <origin xyz="$(arg kinect_xyz)" rpy="$(arg kinect_rpy)" />
+      <parent link="sensor_arch_mount_link"/>
+      <child link="camera_link"/>
     </joint>
-    <!-- IMU Link is the standard mounting position for the UM6 IMU.-->
-    <!-- Can be modified with environment variables in /etc/ros/setup.bash -->
-    <link name="imu_link" />
-    <joint name="imu_joint" type="fixed">
-        <origin rpy="0 -1.5708 3.1416" xyz="0.19 0 0.149" />
-        <parent link="base_link" />
-        <child link="imu_link" />
-    </joint>
-    <gazebo reference="imu_link" />
-    <link name="front_left_wheel_link">
-        <inertial>
-            <mass value="2.637" />
-            <origin xyz="0 0 0" />
-            <inertia ixx="0.02467" ixy="0" ixz="0" iyy="0.04411" iyz="0" izz="0.02467" />
-        </inertial>
-        <visual>
-            <origin rpy="0 0 0" xyz="0 0 0" />
-            <geometry>
-                <mesh filename="package://husky_description/meshes/wheel.dae" />
-            </geometry>
-        </visual>
-        <collision>
-            <origin rpy="1.570795 0 0" xyz="0 0 0" />
-            <geometry>
-                <cylinder length="0.1143" radius="0.1651" />
-            </geometry>
-        </collision>
-    </link>
-    <gazebo reference="front_left_wheel_link">
-        <mu1 value="1.0" />
-        <mu2 value="1.0" />
-        <kp value="10000000.0" />
-        <kd value="1.0" />
-        <fdir1 value="1 0 0" />
-    </gazebo>
-    <joint name="front_left_wheel" type="continuous">
-        <parent link="base_link" />
-        <child link="front_left_wheel_link" />
-        <origin rpy="0 0 0" xyz="0.256 0.2854 0.03282" />
-        <axis rpy="0 0 0" xyz="0 1 0" />
-    </joint>
-    <transmission name="front_left_wheel_trans" type="SimpleTransmission">
-        <type>transmission_interface/SimpleTransmission</type>
-        <actuator name="front_left_wheel_motor">
-            <mechanicalReduction>1</mechanicalReduction>
-        </actuator>
-        <joint name="front_left_wheel">
-            <hardwareInterface>hardware_interface/VelocityJointInterface</hardwareInterface>
-        </joint>
-    </transmission>
-    <link name="front_right_wheel_link">
-        <inertial>
-            <mass value="2.637" />
-            <origin xyz="0 0 0" />
-            <inertia ixx="0.02467" ixy="0" ixz="0" iyy="0.04411" iyz="0" izz="0.02467" />
-        </inertial>
-        <visual>
-            <origin rpy="0 0 0" xyz="0 0 0" />
-            <geometry>
-                <mesh filename="package://husky_description/meshes/wheel.dae" />
-            </geometry>
-        </visual>
-        <collision>
-            <origin rpy="1.570795 0 0" xyz="0 0 0" />
-            <geometry>
-                <cylinder length="0.1143" radius="0.1651" />
-            </geometry>
-        </collision>
-    </link>
-    <gazebo reference="front_right_wheel_link">
-        <mu1 value="1.0" />
-        <mu2 value="1.0" />
-        <kp value="10000000.0" />
-        <kd value="1.0" />
-        <fdir1 value="1 0 0" />
-    </gazebo>
-    <joint name="front_right_wheel" type="continuous">
-        <parent link="base_link" />
-        <child link="front_right_wheel_link" />
-        <origin rpy="0 0 0" xyz="0.256 -0.2854 0.03282" />
-        <axis rpy="0 0 0" xyz="0 1 0" />
-    </joint>
-    <transmission name="front_right_wheel_trans" type="SimpleTransmission">
-        <type>transmission_interface/SimpleTransmission</type>
-        <actuator name="front_right_wheel_motor">
-            <mechanicalReduction>1</mechanicalReduction>
-        </actuator>
-        <joint name="front_right_wheel">
-            <hardwareInterface>hardware_interface/VelocityJointInterface</hardwareInterface>
-        </joint>
-    </transmission>
-    <link name="rear_left_wheel_link">
-        <inertial>
-            <mass value="2.637" />
-            <origin xyz="0 0 0" />
-            <inertia ixx="0.02467" ixy="0" ixz="0" iyy="0.04411" iyz="0" izz="0.02467" />
-        </inertial>
-        <visual>
-            <origin rpy="0 0 0" xyz="0 0 0" />
-            <geometry>
-                <mesh filename="package://husky_description/meshes/wheel.dae" />
-            </geometry>
-        </visual>
-        <collision>
-            <origin rpy="1.570795 0 0" xyz="0 0 0" />
-            <geometry>
-                <cylinder length="0.1143" radius="0.1651" />
-            </geometry>
-        </collision>
-    </link>
-    <gazebo reference="rear_left_wheel_link">
-        <mu1 value="1.0" />
-        <mu2 value="1.0" />
-        <kp value="10000000.0" />
-        <kd value="1.0" />
-        <fdir1 value="1 0 0" />
-    </gazebo>
-    <joint name="rear_left_wheel" type="continuous">
-        <parent link="base_link" />
-        <child link="rear_left_wheel_link" />
-        <origin rpy="0 0 0" xyz="-0.256 0.2854 0.03282" />
-        <axis rpy="0 0 0" xyz="0 1 0" />
-    </joint>
-    <transmission name="rear_left_wheel_trans" type="SimpleTransmission">
-        <type>transmission_interface/SimpleTransmission</type>
-        <actuator name="rear_left_wheel_motor">
-            <mechanicalReduction>1</mechanicalReduction>
-        </actuator>
-        <joint name="rear_left_wheel">
-            <hardwareInterface>hardware_interface/VelocityJointInterface</hardwareInterface>
-        </joint>
-    </transmission>
-    <link name="rear_right_wheel_link">
-        <inertial>
-            <mass value="2.637" />
-            <origin xyz="0 0 0" />
-            <inertia ixx="0.02467" ixy="0" ixz="0" iyy="0.04411" iyz="0" izz="0.02467" />
-        </inertial>
-        <visual>
-            <origin rpy="0 0 0" xyz="0 0 0" />
-            <geometry>
-                <mesh filename="package://husky_description/meshes/wheel.dae" />
-            </geometry>
-        </visual>
-        <collision>
-            <origin rpy="1.570795 0 0" xyz="0 0 0" />
-            <geometry>
-                <cylinder length="0.1143" radius="0.1651" />
-            </geometry>
-        </collision>
-    </link>
-    <gazebo reference="rear_right_wheel_link">
-        <mu1 value="1.0" />
-        <mu2 value="1.0" />
-        <kp value="10000000.0" />
-        <kd value="1.0" />
-        <fdir1 value="1 0 0" />
-    </gazebo>
-    <joint name="rear_right_wheel" type="continuous">
-        <parent link="base_link" />
-        <child link="rear_right_wheel_link" />
-        <origin rpy="0 0 0" xyz="-0.256 -0.2854 0.03282" />
-        <axis rpy="0 0 0" xyz="0 1 0" />
-    </joint>
-    <transmission name="rear_right_wheel_trans" type="SimpleTransmission">
-        <type>transmission_interface/SimpleTransmission</type>
-        <actuator name="rear_right_wheel_motor">
-            <mechanicalReduction>1</mechanicalReduction>
-        </actuator>
-        <joint name="rear_right_wheel">
-            <hardwareInterface>hardware_interface/VelocityJointInterface</hardwareInterface>
-        </joint>
-    </transmission>
-    <!-- Spawn Husky chassis -->
-    <link name="top_chassis_link">
-        <visual>
-            <origin rpy="0 0 0" xyz="0 0 0" />
-            <geometry>
-                <mesh filename="package://husky_description/meshes/top_chassis.dae" />
-            </geometry>
-        </visual>
-    </link>
-    <!-- Attach chassis to the robot -->
-    <joint name="top_chassis_joint" type="fixed">
-        <parent link="base_link" />
-        <child link="top_chassis_link" />
-    </joint>
-    <!-- Spawn user rails -->
-    <link name="user_rail_link">
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
File: DynamicMotionPlanning/husky/husky_description/urdf/husky0.urdf.xacro (robot description, xacro)
@@ -22,8 +22,8 @@
 -->
 <robot name="husky" xmlns:xacro="http://ros.org/wiki/xacro">
-  <xacro:arg name="laser_enabled" default="false" />
+  <xacro:arg name="laser_enabled" default="true" />
   <xacro:arg name="laser_xyz" default="$(optenv HUSKY_LMS1XX_XYZ 0.2206 0.0 0.00635)" />
   <xacro:arg name="laser_rpy" default="$(optenv HUSKY_LMS1XX_RPY 0.0 0.0 0.0)" />
-  <xacro:arg name="kinect_enabled" default="false" />
+  <xacro:arg name="kinect_enabled" default="true" />
   <xacro:arg name="kinect_xyz" default="$(optenv HUSKY_KINECT_XYZ 0 0 0)" />
   <xacro:arg name="kinect_rpy" default="$(optenv HUSKY_KINECT_RPY 0 0.18 3.14)" />
@@ -52,6 +52,17 @@
   <!-- Base link is the center of the robot's bottom plate -->
   <link name="world" />
+  <joint name="map_joint" type="fixed">
+          <parent link="world"/>
+          <child link="map" />
+  </joint>
+  <link name="map">
+      <inertial>
+              <mass value="1" />
+              <origin xyz="0.0 0.0 0.0" rpy="0 0 0" />
+              <inertia ixx="0.1" ixy="0.0" ixz="0.0"	iyy="0.1" iyz="0.0" izz="0.1" />
+      </inertial>
+  </link>
   <joint name="odom_joint" type="fixed">
-          <parent link="world"/>
+          <parent link="map"/>
           <child link="odom" />
   </joint>
@@ -225,6 +236,19 @@
     <plugin name="husky" filename="libhusky.so"/>
   </gazebo>
-  <gazebo>
-    <plugin name="planning_scene" filename="libplanning_scene.so"/>
+  <!-- <gazebo>
+    <plugin name="gazebo_ros_control" filename="libgazebo_ros_control.so" />
+  </gazebo> -->
+  <gazebo>
+    <plugin name="planning_scene" filename="libplanning_scene.so" />
+  </gazebo>
+  <gazebo>
+    <plugin name="gazebo_ros_p3d" filename="libgazebo_ros_p3d.so">
+      <alwaysOn>true</alwaysOn>
+      <updateRate>30.0</updateRate>
+      <bodyName>base_link</bodyName>
+      <topicName>ground_truth_pose</topicName>
+      <gaussianNoise>0.0</gaussianNoise>
+      <frameName>world</frameName>
+    </plugin>
   </gazebo>
   <!-- Optional custom includes. -->
